File: STM32_Demo_Base_Board.kicad_sch (KiCad schematic)
At the start: 29 parts

Commit message: project rename
Other:
- note added: "STM32 Demo Base Board"
- title: (none) -> STM32 Demo Base Board
- moved on the sheet: C?, D?, J?, R?, U?
